File: pcb/kbd-display-module/kbd-display-module.kicad_sch (KiCad schematic)
At the start: 83 parts, among them Q1 MMBT3906, Q2 MMBT3906, Q3 MMBT3906, Q4 MMBT3906, Q5 MMBT3906, Q6 MMBT3906, SW1 BTN_0, SW10 BTN_9, SW11 BTN_A, SW12 BTN_B, SW13 BTN_C, SW14 BTN_D, SW15 BTN_E, SW16 BTN_F, SW17 BTN_AD, SW18 BTN_DA, SW19 BTN_PLUS, SW2 BTN_1, SW20 BTN_GO, SW21 BTN_PC, SW22 BTN_RS, SW23 BTN_ST, SW24 Single-Step, SW3 BTN_3, SW4 Tayda-A3959, SW5 BTN_4, SW6 BTN_5, SW7 BTN_7, SW8 BTN_7, SW9 BTN_8, U1 74HC42, U2 Color, U3 BLUE, U4 BLUE, U5 BLUE, U6 BLUE, U7 BLUE, U8 74LVC06, U9 74LVC1G06

Commit message: Add Note regarding component cost.
Parts:
- SW3: value BTN_3 -> BTN_2
- SW4: value Tayda-A3959 -> BTN_3
- SW7: value BTN_7 -> BTN_6
Other:
- note added: "Replace with Alt PKG. 74LVC1G06Z-7 is expensive."
Changed lines of the file:
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@@
 		)
 	)
+	(text "Replace with\nAlt PKG. \n74LVC1G06Z-7\nis expensive."
+		(exclude_from_sim no)
+		(at 67.818 126.746 0)
+		(effects
+			(font
+				(size 1.27 1.27)
+			)
+		)
+	)
 	(text "RS"
 		(exclude_from_sim no)
@@
 			)
 		)
-		(property "Value" "Tayda-A3959"
+		(property "Value" "BTN_3"
 			(at 111.76 144.78 0)
 			(do_not_autoplace yes)
@@
 			)
 		)
-		(property "Value" "BTN_3"
+		(property "Value" "BTN_2"
 			(at 99.06 144.78 0)
 			(do_not_autoplace yes)
@@
 			)
 		)
-		(property "Value" "BTN_7"
+		(property "Value" "BTN_6"
 			(at 152.4 144.78 0)
 			(do_not_autoplace yes)

Commit message: Added assembly notes for future changes.
Other:
- note added: "KiCAD's SOT-23 footfrint needs to go!!!"
- note added: "SW Pads are a little long for Tayda SW. Reduce length."
Changed lines of the file:
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@@
+		)
+	)
+	(text "SW Pads are a little long for Tayda SW. Reduce length."
+		(exclude_from_sim no)
+		(at 189.484 146.05 0)
+		(effects
+			(font
+				(size 1.27 1.27)
+			)
 		)
 	)
@@
 			)
 		)
+	)
+	(text "KiCAD's SOT-23 footfrint needs to go!!!"
+		(exclude_from_sim no)
+		(at 173.482 88.138 0)
+		(effects
+			(font
+				(size 1.27 1.27)
+			)
+		)
