File: pcb/mainboard/mainboard.kicad_pcb (KiCad board)
At the start: 2 copper layers, 137 x 197 mm, 103 parts, among them J1 Expansion, J2 Application, J3 USB_C_Receptacle_PowerOnly_6P, U1 65C816, U10 74LV540, U11 74LV540, U12 74LV540, U13 74LV541, U14 #0131, U2 Control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

Commit message: Add 3D for USB and expansion connectors.
Parts:
- J1: value Expansion -> Untitled
Changed lines of the file:
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@@
 		(embedded_fonts no)
 		(model "${KICAD9_3DMODEL_DIR}/Connector_USB.3dshapes/USB_C_Receptacle_HRO_TYPE-C-31-M-17.step"
+			(hide yes)
 			(offset
 				(xyz 0 0 0)
@@
 			)
 		)
+		(model "${KICAD9_3DMODEL_DIR}/Connector_USB.3dshapes/USB_C_Receptacle_GCT_USB4125-xx-x-0190_6P_TopMnt_Horizontal.step"
+			(offset
+				(xyz 0 0 0)
+			)
+			(scale
+				(xyz 1 1 1)
+			)
+			(rotate
+				(xyz -0 -0 -0)
+			)
+		)
 	)
 	(footprint "Resistor_SMD:R_0603_1608Metric"
@@
 			)
 		)
-		(property "Value" "Expansion"
+		(property "Value" "Untitled"
 			(at 0 1 0)
 			(unlocked yes)
@@
 			(pinfunction "GND")
 			(pintype "input")
+			(thermal_bridge_angle 45)
 		)
 		(pad "A" smd roundrect
@@
 		)
 		(embedded_fonts no)
+		(model "${CUSTOM_3DMODEL_DIR}/Connector-Header.3dshapes/Header-Female-2.54mm-2x22-SMT.step"
+			(offset
+				(xyz 0 -3.81 0)
+			)
+			(scale
+				(xyz 1 1 1)
+			)
+			(rotate
+				(xyz -0 -0 -0)
+			)
+		)
 	)
 	(footprint "LED_SMD:LED_0603_1608Metric"
@@
 			(pinfunction "GND")
 			(pintype "input")
+			(thermal_bridge_angle 45)
 		)
 		(pad "2" smd roundrect
@@
 		)
 		(embedded_fonts no)
+		(model "${CUSTOM_3DMODEL_DIR}/Connector-Header.3dshapes/Header-Female-2.54mm-2x22-SMT.step"
+			(offset
+				(xyz 0 -3.81 0)
+			)
+			(scale
+				(xyz 1 1 1)
+			)
+			(rotate
+				(xyz -0 -0 -0)
+			)
+		)
 	)
 	(footprint "Resistor_SMD:R_0603_1608Metric"
@@
 			(xy 277.5 115.5) (xy 277.5 133) (xy 279.25 133) (xy 279.25 115.5) (xy 280.25 116.25) (xy 280.25 133)
 			(xy 281 133) (xy 287 139) (xy 287 136) (xy 285.5 134.5) (xy 285.5 128.5) (xy 287 130) (xy 287 126)
-			(xy 285.5 124.5) (xy 285.5 118.5) (xy 287 120) (xy 287 120) (xy 284 117) (xy 284 131) (xy 282 129)
-			(xy 282 115) (xy 280 113) (xy 275 113) (xy 270 108)
+			(xy 285.5 124.5) (xy 285.5 118.5) (xy 287 120) (xy 284 117) (xy 284 131) (xy 282 129) (xy 282 115)
+			(xy 280 113) (xy 275 113) (xy 270 108)
 		)
 		(stroke
@@
 	(gr_poly
 		(pts
-			(xy 242.75 244.25) (xy 244.25 245.75) (xy 252.25 245.75) (xy 253.625 244.375) (xy 252.5 243.25) (xy 252.5 243.25)
-			(xy 251.5 244.25)
+			(xy 242.75 244.25) (xy 244.25 245.75) (xy 252.25 245.75) (xy 253.625 244.375) (xy 252.5 243.25) (xy 251.5 244.25)
 		)
 		(stroke
@@
 			(pts
 				(xy 245.25 51.25) (xy 252.25 51.25) (xy 253 52) (xy 258.5 52) (xy 259.25 51.25) (xy 262.5 51.25)
-				(xy 263.5 52.25) (xy 268.25 52.25) (xy 268.25 52.25) (xy 268 52.5) (xy 262 52.5) (xy 261.75 52.25)
-				(xy 249.5 52.25) (xy 249 51.75) (xy 245.75 51.75)
+				(xy 263.5 52.25) (xy 268.25 52.25) (xy 268 52.5) (xy 262 52.5) (xy 261.75 52.25) (xy 249.5 52.25)
+				(xy 249 51.75) (xy 245.75 51.75)
 			)
 		)
@@
 		(polygon
 			(pts
-				(xy 282 131) (xy 287 136) (xy 287 134) (xy 282 129) (xy 270 129) (xy 270 129) (xy 272 131)
+				(xy 282 131) (xy 287 136) (xy 287 134) (xy 282 129) (xy 270 129) (xy 272 131)
 			)
 		)
