File: pcb/mainboard/mainboard.kicad_sch (KiCad schematic)
At the start: 103 parts, among them J1 Expansion, J2 Application, J3 USB_C_Receptacle_PowerOnly_6P, U1 65C816, U10 74LV540, U11 74LV540, U12 74LV540, U13 74LV541, U14 #0131, U2 Control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

Commit message: Final tuning.
Other:
- company: Circuit Monkey -> by Circuit Monkey
- title: KIM-1 Modular Replica -> KIM-1000 Modular Replica of KIM-1
Changed lines of the file:
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@@
 	(paper "A3")
 	(title_block
-		(title "KIM-1 Modular Replica")
+		(title "KIM-1000 Modular Replica of KIM-1")
+		(date "2025-09-09")
 		(rev "A")
-		(company "Circuit Monkey")
+		(company "by Circuit Monkey")
 	)
 	(text "PWR Switch and 3V Regulator"

Commit message: Fix chip reference. Was wrong part number provided.
Parts:
- U13: MPN SN74LV540ARGY -> SN74LV541ARKSR
Changed lines of the file:
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@@
 			)
 		)
-		(property "Datasheet" "http://www.ti.com/lit/gpn/sn74LS540"
+		(property "Datasheet" "http://www.ti.com/lit/gpn/sn74LS541"
 			(at 300.99 215.9 90)
 			(effects
@@
 			)
 		)
-		(property "MPN" "SN74LV540ARGY"
+		(property "MPN" "SN74LV541ARKSR"
 			(at 297.18 217.17 0)
 			(effects
