File: pcb/control-logic-module/control-logic-module.kicad_pcb (KiCad board)
At the start: 2 copper layers, 43 x 29 mm, 47 parts, among them U1 74HC04, U2 74AHC1G00, U3 74AHC1G00, U4 TLC556, U5 74LS145, Y1 8MHz

Commit message: Make some corrections. Bump Rev to B.
Routing:
- net /Ψ~{Φ2}: track 17.5 -> 11.8 mm
- net /ΨΦ2: track 16.0 -> 17.2 mm
- net VCC: track 96.9 -> 96.2 mm
- net /Ψ~{R}/W: track 11.8 -> 11.2 mm
Other:
- board text added: "Rev. B"
- board text added: "Rev. B (2025-09)"
- board text removed: "Rev. A"
- board text removed: "Rev. A (2025-07)"

Commit message: Update and finalize rev-b board.
Routing:
- net /Ψ~{Φ2}: track 11.8 -> 22.2 mm
